File: HW/astrouniboard.kicad_sch (KiCad schematic)
At the start: 136 parts, among them J1 Conn_01x03, J10 Conn_01x04, J2 MC-311D, J3 Conn_01x04, J4 Conn_01x03, J5 Conn_01x04, J6 5.5/2.1 Barell DC2, J7 MC-311D, J8 Conn_01x04, J9 Conn_01x04, U1 ME6231, U10 MPU-6000, U11 CH213K, U12 ME3116, U13 CH213K, U14 CH213K, U4 24AA64T-I/OT, U5 STM32G0B1CBTx, U6 CH334P, U7 USBLC6-2SC6, U8 SHT31A-DIS, Y1 TAXM8M4RDBCCT2T / 8MHz, Y2 TAXM12M4RDBCCT2T / 12MHz

Commit message: hw: upgrade KiCad project to v10 format
Update PCB, schematic, and project files to KiCad 10 format (generator_version 10.0).
Add .kicad_prl local layout rules file. Exclude .history/ backup dir from git.

Co-Authored-By: Claude Sonnet 4.6 <noreply@anthropic.com>
Parts:
- added C57: 2n2, Capacitor_SMD:C_0402_1005Metric, symbol Device:C
- added C58: 100n, Capacitor_SMD:C_0402_1005Metric, symbol Device:C
- D3, D4: footprint LED_SMD:LED_0603_1608Metric -> LED_SMD:LED_0402_1005Metric
- U2, U3: value ~ -> (none)
Connections:
- net DIAG: no longer U5.18 (PA7)
- net DIR2: now also U5.26 (PB14); no longer U5.47 (PB8)
- net EN2: now also U5.25 (PB13); no longer U5.46 (PB7)
- net GND: now also U10.1 (CLKIN), U10.11 (FSYNC), U10.9 (AD0/MISO), C57.2, C58.2
- net STEP2: now also U5.27 (PB15); no longer U5.48 (PB9)
- net at U5.23 (PB11): now also R15.1, RIGHT1.2
- net at U8.5 (VDD), U8.6 (~{RESET}): now also U5.48 (PB9); no longer U5.30 (PC6)
- net at U10.10 (REGOUT): now also C58.1
- net at U10.20 (CPOUT): now also C57.1
- now unconnected: U5.45 (PB6)
