File: HW/astrouniboard.kicad_sch (KiCad schematic)
At the start: 138 parts, among them J1 Conn_01x03, J10 Conn_01x04, J2 MC-311D, J3 Conn_01x04, J4 Conn_01x03, J5 Conn_01x04, J6 5.5/2.1 Barell DC2, J7 MC-311D, J8 Conn_01x04, J9 Conn_01x04, U1 ME6231, U10 MPU-6000, U11 CH213K, U12 ME3116, U13 CH213K, U14 CH213K, U4 24AA64T-I/OT, U5 STM32G0B1CBTx, U6 CH334P, U7 USBLC6-2SC6, U8 SHT31A-DIS, Y1 TAXM8M4RDBCCT2T / 8MHz, Y2 TAXM12M4RDBCCT2T / 12MHz

Commit message: reorg
new HW V2 first comit
Parts:
- removed C53: 100nF, Capacitor_SMD:C_0402_1005Metric, symbol Device:C
- removed JP1, JP2: SolderJumper_2_Open, myLib_SMD:Micro SolderJumper, symbol Jumper:SolderJumper_2_Open
Connections:
- net at H4.1: now also H8.1
- net at H3.1: now also H6.1
- net at H5.1: now also H1.1
- net at H7.1: now also H2.1
Other:
- moved on the sheet: H1, H2, H3, H4, H5, H6, H7, H8, U1
