File: HW/astrouniboard.kicad_pcb_bck.kicad_pcb (KiCad board)
At the start: 2 copper layers, 35 x 42 mm, 129 parts, among them J10 Conn_01x04, J2 MC-311D, J3 Conn_01x04, J4 Conn_01x03, J5 Conn_01x04, J6 5.5/2.1 Barell DC2, J7 MC-311D, J8 Conn_01x04, J9 Conn_01x04, U1 ME6231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

Commit message: reorg
new HW V2 first comit
Parts:
- moved R14 7.30 mm to (88.6, 136.0)
- moved R6 5.41 mm to (76.5, 134.3), turned to 0 degrees
- moved D1 3.71 mm to (76.5, 135.2)
- moved D2 3.50 mm to (88.8, 135.0)
- moved J6 1.62 mm to (85.0, 118.6)
- moved C46 1.26 mm to (87.6, 120.0), turned to 90 degrees
- moved U6 0.70 mm to (80.6, 123.7)
- moved C56 0.46 mm to (82.6, 117.1)
- moved R22 0.08 mm to (90.0, 109.1)
- moved Y2 0.08 mm to (84.5, 124.0)
Connections:
- H1 pad 1: Net-(H1-Pad1) -> unconnected-(H1-Pad1)
- H2 pad 1: Net-(H2-Pad1) -> unconnected-(H2-Pad1)
- H3 pad 1: Net-(H3-Pad1) -> unconnected-(H3-Pad1)
- H4 pad 1: Net-(H4-Pad1) -> unconnected-(H4-Pad1)
- H5 pad 1: Net-(H1-Pad1) -> unconnected-(H5-Pad1)
- H6 pad 1: Net-(H3-Pad1) -> unconnected-(H6-Pad1)
- H7 pad 1: Net-(H2-Pad1) -> unconnected-(H7-Pad1)
- H8 pad 1: Net-(H4-Pad1) -> unconnected-(H8-Pad1)
Routing:
- net +5V: track 49.9 -> 23.9 mm, vias 8 -> 1
- net /DP2: track 13.6 -> 5.73 mm, vias 2 -> 0
- net /DM2: track 13.9 -> 6.57 mm, vias 2 -> 0
- net Net-(U6-XO): track 6.08 -> 0.25 mm
- net Net-(U5-PB4): track 63.6 -> 58.1 mm
- net Net-(U6-XI): track 4.42 -> 0.04 mm
- net +3.3V: track 150.5 -> 147.1 mm
- net Net-(D2-K): track 2.85 -> 0.00 mm
- net Net-(D1-K): track 2.38 -> 0.00 mm
- net Net-(U5-PB12): track 35.0 -> 37.0 mm
- net Net-(D23-K): track 8.68 -> 10.4 mm
- net /DP: track 40.6 -> 39.2 mm
- net GND: track 6.14 -> 7.55 mm, vias 251 -> 233
- net Net-(J5-Pin_1): track 26.8 -> 28.2 mm
- net /DM: track 39.9 -> 38.7 mm
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Other:
- board text added: "V_DRIVE"
